File: PCB/PiicoDev-Pressure-Sensor-MS5637.kicad_pcb (KiCad board)
At the start: 2 copper layers, 25.4 x 25.4 mm, 19 parts, among them J1 , J2 , J3 Conn_PiicoDev_header_01x04_Ma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, U1 MS5637

Commit message: Change 4k7 resistors to 10k
Parts:
- R1, R3, R4: value 4k7 -> 10k
